File: hardware/handoff.kicad_pcb (KiCad board)
At the start: 2 copper layers, 40 x 62 mm, 65 parts, among them J1 BAT XH-2, J2 PAD JST-XH 2p, J3 LED JST-XH 4p / 5mm RGB, J5 CHG XH-2, SW1 SS-12F23G5, SW2 TACT 6x6, U1 Raspberry Pi Pico 2 W, U2 MCP6292-E/MS

Commit message: Move the breakout pads out of the AFE channel, and route the amplifier
The ten expansion pads sat inboard of their pin rows, one hop into the 10 mm
channel under the Pico, which is what over-subscribed it: R2's pad stopped
0.225 mm short of U2 pin 1 and there was no routing lane at all.

Outboard, between each pin row and the wall, they cost the channel nothing and
each pad is still a single hop from its own pin. The channel is the full
16.2 mm between the pin rows and the AFE columns open to x 15.6 and 24.4.

R2 moves 2 mm toward the hand so pins 1 and 2 have a slot to escape into - the
1 MOhm island grows 6.4 to 8.4 mm for it. The ammeter cluster moves to the
board edge because x 32.3 is now a breakout column. The thumb stubs run on the
bottom face so the top lane at x 9.7 stays clear for C4.

Both gain stages, the island, the VREF bus, the interstage cap and the ADC
filter now route. 27 unconnected items down to 17, with no shorts, no
crossings and no clearance violations; parity still 0. What is left is the
elbow jumper block and AFE_3V3's exit from the channel, written up in the
README.

Co-Authored-By: Claude Opus 5 <noreply@anthropic.com>
Parts:
- moved JP5 5.60 mm to (37.9, 47.7)
- moved TP11 5.60 mm to (37.9, 45.0)
- moved TP8 5.60 mm to (37.9, 50.4)
- moved E10 5.08 mm to (31.4, 55.5)
- moved E3 5.08 mm to (31.4, 60.6)
- moved E4 5.08 mm to (31.4, 58.1)
- moved E5 5.08 mm to (31.4, 47.9)
- moved E6 5.08 mm to (31.4, 45.4)
- moved E1 5.06 mm to (8.60, 50.4)
- moved E2 5.06 mm to (8.60, 35.2)
- moved E7 5.06 mm to (8.60, 25.0)
- moved E8 5.06 mm to (8.60, 27.6)
- moved E9 5.06 mm to (8.60, 40.3)
- moved R2 2.00 mm to (19.7, 24.0)
- moved C1 1.10 mm to (15.6, 41.8)
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Routing:
- net Net-(JP6-A): track 0.00 -> 65.8 mm, vias 0 -> 2
- net /OUT1: track 0.00 -> 53.2 mm, vias 0 -> 1
- net VREF: track 18.1 -> 35.6 mm, vias 0 -> 2
- net Net-(U2A--): track 0.00 -> 16.0 mm
- net Net-(JP1-A): track 0.00 -> 12.9 mm, vias 0 -> 1
- net /ADC0: track 0.00 -> 12.3 mm
- net Net-(JP3-C): track 0.00 -> 8.65 mm, vias 0 -> 1
- net VSYS: track 34.7 -> 39.7 mm
- net /AFE_3V3: track 0.00 -> 4.52 mm
- net Net-(D1-K): track 9.12 -> 13.3 mm
- net Net-(U2B--): track 11.2 -> 14.5 mm
- net Net-(U2A-+): track 5.32 -> 8.41 mm
- net GND: track 0.00 -> 2.30 mm, vias 0 -> 4
- net Net-(JP7-B): track 22.7 -> 20.8 mm
- net Net-(JP3-B): track 5.22 -> 6.06 mm
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
Commit message: Remove all thirteen test pads, and re-lay the elbow block
Each test pad sat on the same net as a solder-jumper pad, a connector pin or a
Pico header pin a couple of millimetres away, and this board is probed with a
meter or a scope tip rather than a clip, so every one of them was a duplicate
occupying through-hole space in the two places the board had none.

Five were in the elbow jumper block, which had eleven parts in 12 x 13 mm:
three gaps of 0.9 mm across it and none at all down the sides. With six parts
it re-lays as two columns 2.96 mm apart with a corridor between them. R10 is
flipped end for end so its two links become single hops instead of crossing.

65 footprints to 52, and 17 unconnected items to 3. The three that remain are
all behind OUT1's descent on the right-hand side; the README says what would
clear them. No shorts, no crossings, no clearance violations, parity still 0.

Costs JP5's ammeter position: board current now means holding a meter across
JP5's own 1 x 0.5 mm pads.

Co-Authored-By: Claude Opus 5 <noreply@anthropic.com>
Parts:
- removed TP1: PAD, TestPoint:TestPoint_Pad_D1.5mm
- removed TP10: BAT+, TestPoint:TestPoint_Pad_D1.5mm
- removed TP11: D1_K, TestPoint:TestPoint_Pad_D1.5mm
- removed TP12: RX_IN, TestPoint:TestPoint_Pad_D1.5mm
- removed TP13, TP7: GND, TestPoint:TestPoint_Pad_D1.5mm
- removed TP2: OUT1, TestPoint:TestPoint_Pad_D1.5mm
- removed TP3: AFE_OUT, TestPoint:TestPoint_Pad_D1.5mm
- removed TP4: ADC0, TestPoint:TestPoint_Pad_D1.5mm
- removed TP5: VREF, TestPoint:TestPoint_Pad_D1.5mm
- removed TP6: AFE_3V3, TestPoint:TestPoint_Pad_D1.5mm
- removed TP8: VSYS, TestPoint:TestPoint_Pad_D1.5mm
- removed TP9: GP11 TX, TestPoint:TestPoint_Pad_D1.5mm
- moved JP3 2.57 mm to (23.5, 50.0)
- moved JP1 2.00 mm to (23.5, 54.0)
- moved JP6 1.50 mm to (16.5, 54.0)
- moved JP4 1.00 mm to (16.5, 50.0), turned to 0 degrees
- turned R10 to -90 degrees
Routing:
- net +3V3: track 2.52 -> 74.0 mm, vias 0 -> 1
- net VREF: track 35.6 -> 52.0 mm, vias 2 -> 3
- net /OUT1: track 53.2 -> 37.6 mm
- net /ADC0: track 12.3 -> 27.1 mm, vias 0 -> 1
- net Net-(JP7-B): track 20.8 -> 14.3 mm
- net Net-(JP3-C): track 8.65 -> 3.31 mm
- net Net-(JP1-A): track 12.9 -> 8.60 mm
- net Net-(D1-K): track 13.3 -> 9.07 mm
- net Net-(JP6-A): track 65.8 -> 69.9 mm, vias 2 -> 1
- net /PAD: track 28.7 -> 24.9 mm
- net /BAT+: track 56.5 -> 53.0 mm
- net /AFE_3V3: track 4.52 -> 6.45 mm, vias 0 -> 1
- net VSYS: track 39.7 -> 39.0 mm

Commit message: Route the last three connections: OUT1 dives under the channel
OUT1 leaves the AFE down the outermost east lane and crosses to C1 on
the bottom face, between BAT+ and SW_OUT, so nothing on the top face
crosses the channel between the amplifier and the elbow. AFE_3V3 and
OUT2 take the two lanes inside it. 0 unrouted, 0 DRC errors.

Co-Authored-By: Claude Opus 5 <noreply@anthropic.com>
Routing:
- net /AFE_3V3: track 6.45 -> 65.3 mm, vias 1 -> 4
- net Net-(JP3-B): track 6.06 -> 21.5 mm, vias 0 -> 1
- net /OUT1: track 37.6 -> 41.3 mm, vias 1 -> 4
- net VREF: track 52.0 -> 49.5 mm, vias 3 -> 1
