File: hardware/handoff.kicad_sch (KiCad schematic)
At the start: 68 parts, among them J1 BAT XH-2, J2 PAD JST-XH 2p, J3 LED JST-XH 4p / 5mm RGB, J5 CHG XH-2, J6 MOT 1x02 2.54, M1 1034 coin 10mm 3V, Q1 AO3400A, SW1 SS-12F23G5, SW2 TACT 6x6, U1 Raspberry Pi Pico 2 W, U2 MCP6292-E/MS

Commit message: Remove E1-E10, shrink the boss to 6 mm, and untangle the elbow
The board came in with 51 DRC errors. The previous session had been asked to
move D3 to the SS220F (SMB) like D1, and there was nowhere to put it: the SMB
took TP2 and TP3's spot beside J6, TP2 and TP3 were pushed out through two
gaps in the Pico's pin row to the little-finger wall, and there they landed on
top of the breakout pads. Four vias and two shorted pads to make room for one
diode. Take the space back instead of routing round the lack of it.

E1-E10 go. Ten through-hole pads on nets nothing uses, a column down each
wall, three of them (GP0, GP1, GND) sitting inside H4's boss for three
sessions. Gone from the schematic, the board, the DRU rule and the parts
list; the eight Pico pins they broke out are no-connect again, which is what
the sheet should say about a pin that goes nowhere. The Pico is socketed -
its own header is the breakout, and always was.

The boss is 6 mm, not 8. Six is enough to hold the 5 mm brass insert with a
wall round it; eight reached 4 mm in from two edges at once and was the only
reason each screw sat 4.5 mm from its corner. Hole position is derived now
rather than written out four times - BOSS_R + BOSS_EDGE from both edges - so
the boss keeps the same half-millimetre of wall and the screws move to
(3.5, 3.5) and its three mirrors. The footprint's name carries the diameter,
so a board built against a stale footprint cannot claim a keep-out it has
not got. The enclosure's printed bosses have to follow: 1 mm out
diagonally, 2 mm smaller.

Test pads are placed last now, into space the layout has already settled.
TP2 and TP3 sit ON their own net's existing lane, each replacing a via that
was there anyway, so neither costs a track, a corner or a pin-row crossing:
TP2 at (18.8, 54.0) on JP1's ADC0 pad row, TP3 at (21.0, 48.6) on OUT1's own
change of face into JP3. ADC0's lane moves to x 19.8 and OUT1's steps 0.8 mm
west to give TP3 its pad, which also has to clear JP3's pin-1 a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
Parts:
- removed E5: GP4 (pin 6), TestPoint:TestPoint_THTPad_D1.5mm_Drill0.7mm, symbol Connector:TestPoint
- removed E8: GP21 (pin 27), TestPoint:TestPoint_THTPad_D1.5mm_Drill0.7mm, symbol Connector:TestPoint
- removed H3: M3, handoff:MountingHole_3.4mm_M3_Boss8mm, symbol Mechanical:MountingHole
- removed JP8: ROLE, Jumper:SolderJumper-2_P1.3mm_Open_RoundedPad1.0x1.5mm, symbol Jumper:SolderJumper_2_Open
- removed M1: 1034 coin 10mm 3V, symbol Motor:Motor_DC
- removed Q1: AO3400A, Package_TO_SOT_SMD:SOT-23, symbol Transistor_FET:AO3400A
- removed R16: 100, Resistor_SMD:R_0603_1608Metric_Pad0.98x0.95mm_HandSolder, symbol Device:R
- removed R17: 100k, Resistor_SMD:R_0603_1608Metric_Pad0.98x0.95mm_HandSolder, symbol Device:R
- removed TP1: GND, TestPoint:TestPoint_THTPad_D1.5mm_Drill0.7mm, symbol Connector:TestPoint
- removed TP2: ADC0, TestPoint:TestPoint_THTPad_D1.5mm_Drill0.7mm, symbol Connector:TestPoint
- removed TP4: VREF, TestPoint:TestPoint_THTPad_D1.5mm_Drill0.7mm, symbol Connector:TestPoint
- added R15: 10k, Resistor_SMD:R_0603_1608Metric_Pad0.98x0.95mm_HandSolder, symbol Device:R
- D3: value 1N5819W -> SS220F; footprint Diode_SMD:D_SOD-123 -> Diode_SMD:D_SMB
- H1, H4: footprint handoff:MountingHole_3.4mm_M3_Boss8mm -> handoff:MountingHole_3.4mm_M3_Boss6mm
- H2: renamed from TP5; value PAD -> M3; footprint TestPoint:TestPoint_THTPad_D1.5mm_Drill0.7mm -> handoff:MountingHole_3.4mm_M3_Boss6mm; symbol Connector:TestPoint -> Mechanical:MountingHole
- H3: renamed from TP6; value VSYS -> M3; footprint TestPoint:TestPoint_THTPad_D1.5mm_Drill0.7mm -> handoff:MountingHole_3.4mm_M3_Boss6mm; symbol Connector:TestPoint -> Mechanical:MountingHole
- JP8: renamed from TP3; value OUT1 -> ROLE; footprint TestPoint:TestPoint_THTPad_D1.5mm_Drill0.7mm -> Jumper:SolderJumper-2_P1.3mm_Open_RoundedPad1.0x1.5mm; symbol Connector:TestPoint -> Jumper:SolderJumper_2_Open
- M1: renamed from H2; value M3 -> 1034 coin 10mm 3V; footprint handoff:MountingHole_3.4mm_M3_Boss8mm -> (none); symbol Mechanical:MountingHole -> Motor:Motor_DC; now in the parts list
- Q1: renamed from TP7; value D1_K -> AO3400A; footprint TestPoint:TestPoint_THTPad_D1.5mm_Drill0.7mm -> Package_TO_SOT_SMD:SOT-23; symbol Connector:TestPoint -> Transistor_FET:AO3400A; now in the parts list
- R16: renamed from TP8; value AFE_3V3 -> 100; footprint TestPoint:TestPoint_THTPad_D1.5mm_Drill0.7mm -> Resistor_SMD:R_0603_1608Metric_Pad0.98x0.95mm_HandSolder; symbol Connector:TestPoint -> Device:R; now in the parts list
- R17: renamed from R15; value 10k -> 100k
- TP1: renamed from E1; value 3V3 (pin 36) -> GND
- TP2: renamed from E2; value RUN (pin 30) -> ADC0
- TP3: renamed from E3; value GP3 (pin 5) -> OUT1
- TP4: renamed from E4; value GP22 (pin 29) -> VREF
- TP5: renamed from E6; value GP5 (pin 7) -> PAD
- TP6: renamed from E7; value GP20 (pin 26) -> VSYS
- TP7: renamed from E9; value GP27 (pin 32) -> D1_K
- TP8: renamed from E10; value GND (pin 8) -> AFE_3V3
Connections:
- net +3V3: now also R15.1; no longer R17.1, TP1.1
- net ADC0: now also TP2.1
- net AFE_3V3: now also TP8.1; no longer R16.1
- net BTN: now also R15.2; no longer R17.2
- net D1_K: now also TP7.1; no longer Q1.1
- net GND: now also JP8.2 (B), Q1.2 (S), R17.2, TP1.1; no longer TP8.1
- net MOT_DRV: now also R16.1
- net MOT_SW: now also M1.2 (-), Q1.3 (D)
- net OUT1: now also TP3.1; no longer JP8.1
- net PAD: now also TP5.1; no longer H2.1
- net ROLE: now also JP8.1 (A)
- net VREF: now also TP4.1
- net VSYS: now also M1.1 (+), TP6.1; no longer H3.1
- net GP20: no longer names the net of U1.26 (GPIO20)
- net GP20: no longer TP6.1
- net GP21: no longer names the net of U1.27 (GPIO21)
- net GP22: no longer names the net of U1.29 (GPIO22)
- net GP22: no longer TP4.1
- net GP27_ADC1: no longer names the net of U1.32 (GPIO27_ADC1)
- net GP27_ADC1: no longer TP7.1
- net GP3: no longer names the net of U1.5 (GPIO3)
- net GP3: no longer TP3.1
- net GP4: no longer names the net of U1.6 (GPIO4)
- net GP5: no longer names the net of U1.7 (GPIO5)
- net GP5: no longer TP5.1
- net RUN: no longer names the net of U1.30 (RUN)
- net RUN: no longer TP2.1
- new net: Q1.1 (G), R16.2, R17.1
- no-connect marks 15 -> 23
Other:
- note added: "(M1 drawn for reference: the motor whose leads go into J6, not a board component.)"
- note added: "D3 is the flyback path: without it the motor's collapse drives Q1's drain well above VSYS"
- note added: "H1-H4: 3.4 mm unplated, 6 mm boss keep-out, one per corner, not tied to GND"
- note added: "Through-hole, 1.5 mm pad / 0.7 mm drill: a wire solders in."
- note added: "at every turn-off. Firmware: GP28 high runs the motor - never during an RX window."
- note removed: "(M1 drawn for reference: it is the motor whose leads go into J6, not a board component.) D3 is the flyback path: without it the"
- note removed: "E1-E10 EXPANSION — one breakout pad inboard of its own Pico pin"
- note removed: "H1-H4: 3.4 mm unplated, 8 mm boss keep-out, one per corner, not tied to GND"
- note removed: "The spare ADC (GP27) is deliberate: a second analogue path is the likeliest hack this board will need."
- note removed: "Through-hole, 1.5 mm pad / 0.7 mm drill: a wire solders in. RUN to GND is a reset."
- note removed: "motor's collapse drives Q1's drain well above VSYS at every turn-off. Firmware: GP28 high runs the motor - never during an RX window."
- moved on the sheet: R17, TP7, TP8

Commit message: Move every passive to 0603 and D1/D3 to the PMEG3020ER-TP (SOD-123FL)
The 12 Sep order: R1-R3, R9, C1-C3, C6 from 1206 and C4/C5 from 0805 to 0603;
both Schottkys from the SS220F (SMB) to the Tech Public PMEG3020ER-TP, 40 V
2 A, in SOD-123FL - not the Nexperia part of the same number. KiCad has no
SOD-123FL, so gen_sod123fl_footprint.py writes one from the outline drawing
and proves it on a test board. No net changes; EXPECTED_NETS is untouched.

What the pad shift broke, all found by the checks: C1 landed on the VREF bus
it used to straddle (origin now on the bus, OUT1's corridor derived from it);
the AFE pocket's exit between R3's pads closed under VREF's 45 (VREF enters
R3.2 flat now); C6 could not straddle BAT+ (stands under JP2 instead); R3's
old pad centre became a bare right angle. R2 moves 1 mm toward U2 and the
1 MOhm island is 8.5 mm, written entirely against pads. Both diodes needed no
route change. Pours: top 1611 -> 1630 mm2, bottom 1155 -> 1179. D1's cathode
bar is on silk again.

gen_bom.py now derives bom.csv's Package column instead of it being typed in;
gen_schematic.py calls it. README: parts table, D1 deviation (0.4 V, and the
GP29 correction now agrees with it), the 10 uF paragraph, one-package
statement, and a session log with the C0G / 25 V / R2-R3 ESD reasoning.

Co-Authored-By: Claude Opus 5 <noreply@anthropic.com>
Parts:
- C1, C2, C3, C6: footprint Capacitor_SMD:C_1206_3216Metric_Pad1.33x1.80mm_HandSolder -> Capacitor_SMD:C_0603_1608Metric_Pad1.08x0.95mm_HandSolder
- C4, C5: value 10uF 100V -> 10uF 25V; footprint Capacitor_SMD:C_0805_2012Metric_Pad1.18x1.45mm_HandSolder -> Capacitor_SMD:C_0603_1608Metric_Pad1.08x0.95mm_HandSolder
- D1, D3: value SS220F -> PMEG3020ER-TP; footprint Diode_SMD:D_SMB -> handoff:D_SOD-123FL
- R1, R2, R3, R9: footprint Resistor_SMD:R_1206_3216Metric_Pad1.30x1.75mm_HandSolder -> Resistor_SMD:R_0603_1608Metric_Pad0.98x0.95mm_HandSolder
Other:
- note added: "TP8 is new: C4 and C5 are 0603 MLCC now, so the through-hole + lead that used to be the AFE_3V3 probe point is gone."
- note removed: "TP8 is new: C4 and C5 are 0805 MLCC now, so the through-hole + lead that used to be the AFE_3V3 probe point is gone."
Changed lines of the file:
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@@
 		)
 	)
-	(text "TP8 is new: C4 and C5 are 0805 MLCC now, so the through-hole + lead that used to be the AFE_3V3 probe point is gone."
+	(text "TP8 is new: C4 and C5 are 0603 MLCC now, so the through-hole + lead that used to be the AFE_3V3 probe point is gone."
 		(exclude_from_sim no)
 		(at 190.5000 259.0800 0)
@@
 			)
 		)
-		(property "Value" "SS220F"
+		(property "Value" "PMEG3020ER-TP"
 			(at 83.8200 34.2900 0)
 			(effects
@@
 			)
 		)
-		(property "Footprint" "Diode_SMD:D_SMB"
+		(property "Footprint" "handoff:D_SOD-123FL"
 			(at 83.8200 30.4800 0)
 			(effects
@@
 			)
 		)
-		(property "Description" "VSYS OR-ing / reverse polarity, Schottky 200 V 2 A, SMB"
+		(property "Description" "VSYS OR-ing / reverse polarity, Schottky 40 V 2 A, SOD-123FL (Tech Public, not Nexperia)"
 			(at 83.8200 30.4800 0)
 			(effects
@@
 			)
 		)
-		(property "Value" "10uF 100V"
+		(property "Value" "10uF 25V"
 			(at 169.6400 52.3000 0)
 			(effects
@@
 			)
 		)
-		(property "Footprint" "Capacitor_SMD:C_0805_2012Metric_Pad1.18x1.45mm_HandSolder"
+		(property "Footprint" "Capacitor_SMD:C_0603_1608Metric_Pad1.08x0.95mm_HandSolder"
 			(at 167.6400 50.8000 0)
 			(effects
@@
 			)
 		)
-		(property "Description" "VREF hold-up, 0805 MLCC"
+		(property "Description" "VREF hold-up, X5R 0603"
 			(at 167.6400 50.8000 0)
 			(effects
@@
 			)
 		)
-		(property "Footprint" "Capacitor_SMD:C_1206_3216Metric_Pad1.33x1.80mm_HandSolder"
+		(property "Footprint" "Capacitor_SMD:C_0603_1608Metric_Pad1.08x0.95mm_HandSolder"
 			(at 279.4000 45.7200 0)
 			(effects
@@
 			)
 		)
-		(property "Value" "10uF 100V"
+		(property "Value" "10uF 25V"
 			(at 294.1000 47.2200 0)
 			(effects
@@
 			)
 		)
-		(property "Footprint" "Capacitor_SMD:C_0805_2012Metric_Pad1.18x1.45mm_HandSolder"
+		(property "Footprint" "Capacitor_SMD:C_0603_1608Metric_Pad1.08x0.95mm_HandSolder"
 			(at 292.1000 45.7200 0)
 			(effects
@@
 			)
 		)
-		(property "Description" "U2 bulk decoupling against the Pico SMPS, 0805 MLCC"
+		(property "Description" "U2 bulk decoupling against the Pico SMPS, X5R 0603"
 			(at 292.1000 45.7200 0)
 			(effects
@@
 			)
 		)
-		(property "Footprint" "Resistor_SMD:R_1206_3216Metric_Pad1.30x1.75mm_HandSolder"
+		(property "Footprint" "Resistor_SMD:R_0603_1608Metric_Pad0.98x0.95mm_HandSolder"
 			(at 170.1800 111.7600 0)
 			(effects
@@
 			)
 		)
-		(property "Footprint" "Capacitor_SMD:C_1206_3216Metric_Pad1.33x1.80mm_HandSolder"
+		(property "Footprint" "Capacitor_SMD:C_0603_1608Metric_Pad1.08x0.95mm_HandSolder"
 			(at 149.8600 101.6000 0)
 			(effects
@@
 			)
 		)
-		(property "Footprint" "Resistor_SMD:R_1206_3216Metric_Pad1.30x1.75mm_HandSolder"
+		(property "Footprint" "Resistor_SMD:R_0603_1608Metric_Pad0.98x0.95mm_HandSolder"
 			(at 215.9000 127.0000 0)
 			(effects
@@
 			)
 		)
-		(property "Footprint" "Resistor_SMD:R_1206_3216Metric_Pad1.30x1.75mm_HandSolder"
+		(property "Footprint" "Resistor_SMD:R_0603_1608Metric_Pad0.98x0.95mm_HandSolder"
 			(at 231.1400 139.7000 0)
 			(effects
@@
 			)
 		)
-		(property "Footprint" "Capacitor_SMD:C_1206_3216Metric_Pad1.33x1.80mm_HandSolder"
+		(property "Footprint" "Capacitor_SMD:C_0603_1608Metric_Pad1.08x0.95mm_HandSolder"
 			(at 274.3200 129.5400 0)
 			(effects
@@
 			)
 		)
-		(property "Footprint" "Resistor_SMD:R_1206_3216Metric_Pad1.30x1.75mm_HandSolder"
+		(property "Footprint" "Resistor_SMD:R_0603_1608Metric_Pad0.98x0.95mm_HandSolder"
 			(at 328.9300 132.0800 0)
 			(effects
@@
 			)
 		)
-		(property "Footprint" "Capacitor_SMD:C_1206_3216Metric_Pad1.33x1.80mm_HandSolder"
+		(property "Footprint" "Capacitor_SMD:C_0603_1608Metric_Pad1.08x0.95mm_HandSolder"
 			(at 354.3300 139.7000 0)
 			(effects
@@
 			)
 		)
-		(property "Value" "SS220F"
+		(property "Value" "PMEG3020ER-TP"
 			(at 88.9000 255.2700 90)
 			(effects
@@
 			)
 		)
-		(property "Footprint" "Diode_SMD:D_SMB"
+		(property "Footprint" "handoff:D_SOD-123FL"
 			(at 91.4400 255.2700 0)
 			(effects
@@
 			)
 		)
-		(property "Description" "Motor flyback, Schottky 200 V 2 A, SMB"
+		(property "Description" "Motor flyback, Schottky 40 V 2 A, SOD-123FL (Tech Public, not Nexperia)"
 			(at 91.4400 255.2700 0)
 			(effects
